Commit message: [add]添加备份与opendoge新URDF

File: resources/robots/Opendoge_copy/urdf/Opendoge.urdf (robot description, URDF)
Before this commit: robot Opendoge, 17 links, 16 joints
Links:
- link FL_calf: geometry collision mesh filename=../meshes/FL_calf.STL; visual mesh filename=../meshes/FL_calf.STL
- link FL_foot: geometry collision mesh filename=../meshes/FL_foot.STL; visual mesh filename=../meshes/FL_foot.STL
- link FL_hip: geometry collision mesh filename=../meshes/FL_hip.STL; visual mesh filename=../meshes/FL_hip.STL
- link FL_thigh: geometry collision mesh filename=../meshes/FL_thigh.STL; visual mesh filename=../meshes/FL_thigh.STL
- link FR_calf: geometry collision mesh filename=../meshes/FR_calf.STL; visual mesh filename=../meshes/FR_calf.STL
- link FR_foot: geometry collision mesh filename=../meshes/FR_foot.STL; visual mesh filename=../meshes/FR_foot.STL
- link FR_hip: geometry collision mesh filename=../meshes/FR_hip.STL; visual mesh filename=../meshes/FR_hip.STL
- link FR_thigh: geometry collision mesh filename=../meshes/FR_thigh.STL; visual mesh filename=../meshes/FR_thigh.STL
- link RL_calf: geometry collision mesh filename=../meshes/RL_calf.STL; visual mesh filename=../meshes/RL_calf.STL
- link RL_foot: geometry collision mesh filename=../meshes/RL_foot.STL; visual mesh filename=../meshes/RL_foot.STL
- link RL_hip: geometry collision mesh filename=../meshes/RL_hip.STL; visual mesh filename=../meshes/RL_hip.STL
- link RL_thigh: geometry collision mesh filename=../meshes/RL_thigh.STL; visual mesh filename=../meshes/RL_thigh.STL
- link RR_calf: geometry collision mesh filename=../meshes/RR_calf.STL; visual mesh filename=../meshes/RR_calf.STL
- link RR_foot: geometry collision mesh filename=../meshes/RR_foot.STL; visual mesh filename=../meshes/RR_foot.STL
- link RR_hip: geometry collision mesh filename=../meshes/RR_hip.STL; visual mesh filename=../meshes/RR_hip.STL
- link RR_thigh: geometry collision mesh filename=../meshes/RR_thigh.STL; visual mesh filename=../meshes/RR_thigh.STL
- link base_link: geometry collision mesh filename=../meshes/base_link.STL; visual mesh filename=../meshes/base_link.STL
