Commit message: [fix]修正大腿的运动范围

File: resources/robots/Opendoge/urdf/Opendoge.urdf (robot description, URDF)
Before this commit: robot Opendoge, 17 links, 16 joints
Joints:
- joint FL_thigh_joint: limit lower=-0.785 upper=0.785 effort=6 velocity=10.472 -> lower=-0.785 upper=1.134 effort=6 velocity=10.472
- joint FR_thigh_joint: limit lower=-0.785 upper=0.785 effort=6 velocity=10.472 -> lower=-0.785 upper=1.134 effort=6 velocity=10.472
- joint RL_thigh_joint: limit lower=-0.785 upper=0.785 effort=6 velocity=10.472 -> lower=-0.785 upper=1.134 effort=6 velocity=10.472
- joint RR_thigh_joint: limit lower=-0.785 upper=0.785 effort=6 velocity=10.472 -> lower=-0.785 upper=1.134 effort=6 velocity=10.472
